File: pcb/blinkyboard.kicad_pcb (KiCad board)
At the start: 2 copper layers, 83 x 78.5 mm, 18 parts, among them J2 Conn_01x02_Socket, J3 Conn_01x01_Socket, U1 4017, U2 NE555P

Commit message: p
Parts:
- removed J2: Conn_01x02_Socket, Connector_PinHeader_2.54mm:PinHeader_1x02_P2.54mm_Vertical
- removed J3: Conn_01x01_Socket, Connector_PinHeader_2.54mm:PinHeader_1x01_P2.54mm_Vertical
- added D10: LED, LED_THT:LED_D3.0mm, F.Cu at (155.2, 90.4)
- moved U2 99.4 mm to (159.8, 107.9), turned to 90 degrees
- moved C1 91.0 mm to (138.7, 121.9)
- moved D8 89.8 mm to (138.4, 134.6)
- moved RV1 71.8 mm to (152.4, 76.2)
- moved D9 71.2 mm to (175.9, 108.0)
- moved D5 67.7 mm to (101.3, 107.2)
- moved C2 64.0 mm to (114.8, 103.5)
- moved D3 64.0 mm to (147.3, 109.2)
- moved D6 58.8 mm to (129.8, 109.2)
- moved D2 45.5 mm to (122.4, 90.4)
- moved D1 44.5 mm to (138.8, 80.7)
- moved R1 42.2 mm to (121.6, 74.2)
- moved R2 42.2 mm to (121.6, 78.3)
- moved D7 37.4 mm to (161.3, 65.0)
- moved D4 28.0 mm to (116.6, 65.0)
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Connections:
- U1 pad 11: Net-(D9-A) -> Net-(D10-A)
- U1 pad 9: unconnected-(U1-Q8-Pad9) -> Net-(D9-A)
Routing:
- net Net-(D1-K): track 0.00 -> 330.8 mm
- net GND: track 0.00 -> 99.8 mm
- net TR: track 0.00 -> 86.1 mm
- net Net-(D4-A): track 0.00 -> 84.8 mm
- net Net-(U2-DISCH): track 0.00 -> 78.1 mm, vias 0 -> 1
- net +5V: track 0.00 -> 65.9 mm, vias 0 -> 1
- net out: track 0.00 -> 62.1 mm, vias 0 -> 1
- net Net-(D6-A): track 0.00 -> 58.7 mm, vias 0 -> 1
- net Net-(U2-CONT): track 0.00 -> 55.1 mm
- net Net-(D7-A): track 0.00 -> 46.1 mm
- net Net-(D5-A): track 0.00 -> 43.5 mm, vias 0 -> 1
- net Net-(D8-A): track 0.00 -> 37.6 mm
- net Net-(D9-A): track 0.00 -> 36.2 mm
- net Net-(D1-A): track 0.00 -> 22.7 mm, vias 0 -> 1
- net Net-(D3-A): track 0.00 -> 22.2 mm, vias 0 -> 1
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