File: pcb/blinkyboard.kicad_pcb (KiCad board)
At the start: 2 copper layers, 83 x 78.5 mm, 17 parts, among them U1 4017, U2 NE555P

Commit message: blorp
Other:
- outline, holes or cut-outs redrawn

Commit message: zorp
Parts:
- added J1: Conn_01x01_Socket, Connector_PinHeader_2.54mm:PinHeader_1x01_P2.54mm_Vertical, F.Cu at (144.4, 118.0)
- added J2: Conn_01x02_Socket, Connector_PinHeader_2.54mm:PinHeader_1x02_P2.54mm_Vertical, F.Cu at (135.2, 116.9)
- moved C1 2.68 mm to (138.9, 124.6)
Routing:
- net +5V: track 65.9 -> 107.8 mm
- net out: track 62.1 -> 89.5 mm
- net TR: track 86.1 -> 91.0 mm
- net GND: track 99.8 -> 104.4 mm
