File: pcb/blinkyboard.kicad_sch (KiCad schematic)
At the start: 17 parts, among them U1 4017, U2 NE555P

Commit message: zorp
Parts:
- added J1: Conn_01x01_Socket, Connector_PinHeader_2.54mm:PinHeader_1x01_P2.54mm_Vertical, symbol Connector:Conn_01x01_Socket
- added J2: Conn_01x02_Socket, Connector_PinHeader_2.54mm:PinHeader_1x02_P2.54mm_Vertical, symbol Connector:Conn_01x02_Socket
Connections:
- net +5V: now also J2.1 (Pin_1)
- net GND: now also J2.2 (Pin_2)
- net out: now also J1.1 (Pin_1)
